Commit message: feat(phase-1.5): 同步实机硬件边界与部署
统一两种底盘的 DRV8871、MCU 超声波和 v0.2 串口协议，并补齐树莓派生产桥。

增加 Pixhawk/D435i 实机启动与 ARM64 边缘镜像校验，同步完整 BOM、模块边界、部署手册和待上机参数。

File: src/air_ground_car_bringup/urdf/diff_chassis.urdf.xacro (robot description, xacro)
@@ -3,5 +3,5 @@
   <xacro:include
     filename="$(find air_ground_car_bringup)/urdf/car_base.urdf.xacro"/>
-  <xacro:property name="wheel_radius" value="0.033"/>
+  <xacro:property name="wheel_radius" value="0.0325"/>
   <xacro:property name="wheel_width" value="0.026"/>
   <xacro:property name="wheel_separation" value="0.18"/>

File: src/air_ground_car_bringup/urdf/mecanum_chassis.urdf.xacro (robot description, xacro)
@@ -3,5 +3,5 @@
   <xacro:include
     filename="$(find air_ground_car_bringup)/urdf/car_base.urdf.xacro"/>
-  <xacro:property name="wheel_radius" value="0.033"/>
+  <xacro:property name="wheel_radius" value="0.040"/>
   <xacro:property name="wheel_width" value="0.026"/>
   <xacro:property name="wheel_mass" value="0.05"/>

Commit message: feat(phase-1.5): 同步地面车实机参数与安全基线
- 冻结底盘几何、编码器、IMU、云台、RC 与供电参数\n- 实现 STM32 四路超声波捕获及共用 iBUS、RC 安全和正交解码逻辑\n- 拒绝无效 MSPM0 引脚方案并同步部署、测试与交接文档

File: src/air_ground_car_bringup/urdf/diff_chassis.urdf.xacro (robot description, xacro)
@@ -3,7 +3,7 @@
   <xacro:include
     filename="$(find air_ground_car_bringup)/urdf/car_base.urdf.xacro"/>
-  <xacro:property name="wheel_radius" value="0.0325"/>
+  <xacro:property name="wheel_radius" value="0.031"/>
   <xacro:property name="wheel_width" value="0.026"/>
-  <xacro:property name="wheel_separation" value="0.18"/>
+  <xacro:property name="wheel_separation" value="0.166"/>
   <xacro:property name="wheel_mass" value="0.05"/>
   <xacro:property name="caster_radius" value="0.012"/>
@@ -38,5 +38,6 @@
       <origin xyz="0 ${y} ${wheel_radius}" rpy="${-pi / 2.0} 0 0"/>
       <axis xyz="0 0 1"/>
-      <limit effort="5.0" velocity="35.0"/>
+      <!-- 40 rad/s 覆盖供应资料 360±20 RPM 的空载公差上限（约 39.8 rad/s）。 -->
+      <limit effort="5.0" velocity="40.0"/>
       <dynamics damping="0.02" friction="0.0"/>
     </joint>

File: src/air_ground_car_bringup/urdf/mecanum_chassis.urdf.xacro (robot description, xacro)
@@ -3,9 +3,9 @@
   <xacro:include
     filename="$(find air_ground_car_bringup)/urdf/car_base.urdf.xacro"/>
-  <xacro:property name="wheel_radius" value="0.040"/>
+  <xacro:property name="wheel_radius" value="0.0395"/>
   <xacro:property name="wheel_width" value="0.026"/>
   <xacro:property name="wheel_mass" value="0.05"/>
-  <xacro:property name="wheel_x" value="0.10"/>
-  <xacro:property name="wheel_y" value="0.09"/>
+  <xacro:property name="wheel_x" value="0.062"/>
+  <xacro:property name="wheel_y" value="0.083"/>
   <!-- fdir_z is expressed in the wheel collision frame. After the wheel is
        rotated onto its axle, it selects a +/-45 degree ground traction line. -->
@@ -39,5 +39,6 @@
       <origin xyz="${x} ${y} ${wheel_radius}" rpy="${-pi / 2.0} 0 0"/>
       <axis xyz="0 0 1"/>
-      <limit effort="5.0" velocity="35.0"/>
+      <!-- 40 rad/s 覆盖供应资料 360±20 RPM 的空载公差上限（约 39.8 rad/s）。 -->
+      <limit effort="5.0" velocity="40.0"/>
       <dynamics damping="0.02" friction="0.0"/>
     </joint>
